File: Eagle/Power Distribution Board/Battery Board v1.sch (EAGLE design)
At the start: 150 parts, among them IC4 74HC164D, Q3 FDD4141, Q4 FDD4141, Q5 FDD4141, Q6 FDD8447L, Q7 FDD8447L, Q8 FDD8447L, Q9 FDD8447L

Commit message: Reorganise projects & cleanup
Parts:
- removed 5V_FPGA, 5V_IN: 22-23-2021, con-molex:22-23-2021
- removed C1: 0.01uF, rcl:C-EUC0603
- removed C4: 0.1uF, rcl:C-EUC0603
- removed ENCODER1, ENCODER2, ENCODER3, ENCODER4: 22-23-2041, con-molex:22-23-2041
- removed P1, P3: (no value), pinhead:PINHD-2X8
- removed P4: (no value), pinhead:PINHD-2X14
- removed QG1: SM77H, custom:SM77H
- removed R1, R2, R7, R8: 3.3K, rcl:R-EU_R0603
- removed U$1: SN74LVC244, custom:SN74LVC244
Connections:
- removed net GND: 5V_FPGA-2.S, 5V_IN-2.S, C1.2, C4.1, ENCODER1-2.S, ENCODER2-2.S, ENCODER3-2.S, ENCODER4-2.S, P4.1, P4.2, P4.25, P4.26, QG1.GND, U$1.!1OE, U$1.!2OE, U$1.GND
- removed net N$1: P4.14, QG1.OUT
- removed net N$10: ENCODER3-3.S, R1.1, U$1.2A4
- removed net N$11: ENCODER3-4.S, R2.1, U$1.2A3
- removed net N$14: ENCODER4-3.S, R8.1, U$1.2A2
- removed net N$15: ENCODER4-4.S, R7.1, U$1.2A1
- removed net N$16: ENCODER1-3.S, U$1.1A4
- removed net N$17: ENCODER1-4.S, U$1.1A3
- removed net N$18: ENCODER2-3.S, U$1.1A2
- removed net N$19: ENCODER2-4.S, U$1.1A1
- removed net N$2: P4.23, U$1.1Y4
- removed net N$3: P4.21, U$1.1Y2
- removed net N$4: P4.15, U$1.1Y1
- removed net N$5: P4.22, U$1.1Y3
- removed net N$6: P1.4, U$1.2Y4
- removed net N$7: P1.2, U$1.2Y2
- removed net N$8: P1.1, U$1.2Y1
- removed net N$9: P1.3, U$1.2Y3
- removed net VCC3.3: C1.1, C4.2, P4.28, QG1.VCC, U$1.VCC
- removed net VCC5V: 5V_FPGA-1.S, 5V_IN-1.S, ENCODER1-1.S, ENCODER2-1.S, ENCODER3-1.S, ENCODER4-1.S, R1.2, R2.2, R7.2, R8.2
Other:
- moved on the sheet: BAT-1, BAT-2, BAT-CELL-1, BAT-CELL-2, BAT-CELL-3, BAT-CELL-4, BAT-CELL-5, BAT-CELL-6, BAT-CELL-7, BAT-CELL-8, BAT_TEMP-1, BAT_TEMP-2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
