File: Eagle/Elec 2014/Arduino Shield.sch (EAGLE design)
At the start: 63 parts, among them Q1 BC857B, Q2 BC857B, U1 TLC555, U2 SN74HC14PW

Commit message: New servo & aux motor board, updated Arduino shield, new battery board 2014
Parts:
- removed 5V_: 87438-02, con-molex:87438-02
- removed JACK: 87437-0243, custom:87437-0243
- removed Q1, Q2: BC857B, transistor-pnp:MMBTA56-SOT23
- removed RST/LED/COLOR: 87437-0643, custom:87437-0643
- added 5V1: 87438-02, con-molex:87438-02
- added C12, C13, C18, C20, C21, C22, C23, C24: 10uF, rcl:C-EUC0603
- added C14, C25, C26, C27, C28, C29, C30, C31, C32, C33: 47uF, rcl:C-EUC1206
- added C15, C16, C17, C19: 0.1uF, rcl:C-EUC0603
- added CONTROL: 87437-1043, custom:87437-1043
- added IC1: 74LVC1G17DBV, 74xx-little-de:74LVC1G17DBV
- added IC2: 74LVC1G04DCK, 74xx-little-us:74LVC1G04DCK
- added JP1, JP2: (no value), jumper:JP1E
- added R13: 330, rcl:R-EU_R0603
- added R14: 68, rcl:R-EU_R0603
- added R15: 33, rcl:R-EU_R0603
- added R16, R18, R21, R23, R25, R27, R29: 1K, rcl:R-EU_R0603
- added R17, R19, R20, R22, R24, R26, R28: 10K, rcl:R-EU_R0603
- added R30, R31: 1.5K, rcl:R-EU_R0603
- added RBG_SENSOR2, RGB_SENSOR1: 87437-0443, custom:87437-0443
- added U3: SN74HC14PW, custom:SN74HC14PW
- C1, C4, C5, C6, C7, C9: value 0.1uF -> 1uF
- C2: value 0.1uF -> 0.01uF
- R1, R2, R3, R4, R5, R6: value 10K -> 470
- R12: value 10K -> 1K
- SERVOS: value 87437-0443 -> 87437-0843; device custom:87437-0443 -> custom:87437-0843
Connections:
- net N$10 renamed RX1
- net N$11 renamed JACK
- net N$9 renamed TX1
- removed net N$37: Q2.B, R12.1
- removed net N$38: Q1.B, R11.1
- removed net N$46: Q2.C, SONAR_BL.2
- new net BLUE: R15.1, U$1.PWM10
- new net BTN1: U$1.23, U2.3Y
- new net BTN2: U$1.25, U2.4Y
- new net BUT1: CONTROL.7, R16.2, R17.1
- new net BUT2: CONTROL.6, R18.2, R19.1
- new net GREEN: R14.1, U$1.PWM3
- new net N$1: JP1.1, U$1.3.3V
- new net N$10: C18.2, R12.1, U3.6A
- new net N$11: C13.1, R18.1, U2.4A
- new net N$15: CONTROL.5, R15.2
- new net N$16: CONTROL.4, R14.2
- new net N$17: CONTROL.3, R13.2
- new net N$18: SERVOS.8, U$1.31
- new net N$19: R20.1, R21.2, USW2.1
- new net N$20: C20.2, R21.1, U3.5A
- new net N$21: R22.1, R23.2, USW3.1
- new net N$22: C21.2, R23.1, U3.4A
- new net N$23: R24.1, R25.2, USW4.1
- new net N$24: C22.2, R25.1, U3.3A
- new net N$25: R26.1, R27.2, USW5.1
- new net N$26: C23.2, R27.1, U3.2A
- new net N$28: R28.1, R29.2, USW6.1
- new net N$29: C24.2, R29.1, U3.1A
- new net N$7: IC1G$1.O, U$1.RESET
- new net N$8: JP2.1, U$1.5V3
- new net N$9: R11.1, R12.2, USW1.1
- new net RED: R13.1, U$1.PWM2
- new net SCL: RGB_SENSOR1.2, U$1.SCL
- new net SCL1: R31.1, RBG_SENSOR2.2, U$1.SCL1
- new net SDA: RGB_SENSOR1.1, U$1.SDA
- new net SDA1: R30.1, RBG_SENSOR2.1, U$1.SDA1
- net 3.3VCC: now also C15.1, C16.2, C17.2, C19.1, IC1P.VCC, IC2P.VCC, JP1.2, R11.2, R17.2, R19.2, R20.2, R22.2, R24.2, R26.2, R28.2, R30.2, R31.2, RBG_SENSOR2.3, RGB_SENSOR1.3, U3.VCC; no longer Q1.E, Q2.E, U$1.3.3V
- net 5VCC: now also 5V1-1.S, C14.2, C25.2, C26.2, C27.2, C28.2, C29.2, C30.2, C31.2, C32.2, C33.2, JP2.2; no longer 5V_-1.S, U$1.5V3
- net COLOR: now also CONTROL.2; no longer RST/LED/COLOR.2
- net GND: now also 5V1-2.S, C12.2, C13.2, C14.1, C15.2, C16.1, C17.1, C18.1, C19.2, C20.1, C21.1, C22.1, C23.1, C24.1, C25.1, C26.1, C27.1, C28.1, C29.1, C30.1, C31.1, C32.1, C33.1, CONTROL.8, IC1P.GND, IC2P.GND, RBG_SENSOR2.4, RGB_SENSOR1.4, U$1.GND, U$1.GND2, U$1.GND3, U$1.GND5, U2.2A, U3.GND; no longer 5V_-2.S, JACK.2, RST/LED/COLOR.6, U2.3A, U2.4A
- net MOTOR1_BREAK: now also U$1.27; no longer U$1.32
- net MOTOR1_DIR: now also U$1.PWM8; no longer U$1.31
- net MOTOR1_PWM: now also U$1.26; no longer U$1.PWM2
- net MOTOR2_BREAK: now also U$1.29; no longer U$1.34
- net MOTOR2_DIR: now also U$1.PWM9; no longer U$1.33
- net MOTOR2_PWM: now also U$1.28; no longer U$1.PWM3
- net N$12: now also SERVOS.5, U$1.PWM11; no longer RST/LED/COLOR.4, U$1.PWM9
- net N$13: now also SERVOS.6, U$1.PWM12; no longer RST/LED/COLOR.5, U$1.PWM10
- net N$14: now also SERVOS.7, U$1.30; no longer U$1.23, U2.2Y
- net N$2: now also C12.1, R16.1, U2.3A; no longer RST/LED/COLOR.3, U$1.PWM8
- net N$27: now also CONTROL.9; no longer JACK.1
- net N$36: now also IC2A.I; no longer R11.2, R12.2
- net N$44: now also U$1.38; no longer U$1.35
- net N$45: now also IC2A.O, SONAR_BL.2; no longer Q1.C
- net N$47: now also U$1.39; no longer U$1.36
- net N$48: now also U$1.40; no longer U$1.37
- net N$49: now also U$1.41; no longer U$1.38
- net N$50: now also U$1.42; no longer U$1.39
- net N$51: now also U$1.43; no longer U$1.40
- net N$52: now also U$1.44; no longer U$1.41
- net N$53: now also U$1.45; no longer U$1.42
- net N$54: now also U$1.46; no longer U$1.43
- net N$55: now also U$1.47; no longer U$1.44
- net N$56: now also U$1.48; no longer U$1.45
- net N$57: now also U$1.49; no longer U$1.46
- net N$58: now also U$1.50; no longer U$1.47
- net N$59: now also U$1.51; no longer U$1.48
- net N$60: now also U$1.52; no longer U$1.49
- net N$61: now also U$1.53; no longer U$1.50
- net N$71: now also IC1G$1.I; no longer U2.2A
- net RST: now also CONTROL.1; no longer RST/LED/COLOR.1
- net USW1: now also U$1.34, U3.1Y; no longer U$1.25, USW1.1
- net USW2: now also U$1.33, U3.2Y; no longer U$1.26, USW2.1
- net USW3: now also U$1.32, U3.3Y; no longer U$1.27, USW3.1
- net USW4: now also U$1.37, U3.4Y; no longer U$1.28, USW4.1
- net USW5: now also U$1.36, U3.5Y; no longer U$1.29, USW5.1
- net USW6: now also U$1.35, U3.6Y; no longer U$1.30, USW6.1
Other:
- moved on the sheet: 12VIN-1, 12VIN-2, 3.3V-1, 3.3V-2, C10, C11, FPGA, MOTORS, R10, R11, R12, R7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

Commit message: Small fixes after testing cards
Parts:
- C2: value 0.01uF -> 0.1uF
Connections:
- net MOTOR1_BREAK: now also MOTORS.6, U$1.28; no longer MOTORS.3, U$1.27
- net MOTOR1_DIR: now also MOTORS.7, U$1.PWM9; no longer MOTORS.2, U$1.PWM8
- net MOTOR1_PWM: now also MOTORS.8, U$1.29; no longer MOTORS.1, U$1.26
- net MOTOR2_BREAK: now also MOTORS.1, U$1.26; no longer MOTORS.8, U$1.29
- net MOTOR2_DIR: now also MOTORS.2, U$1.PWM8; no longer MOTORS.7, U$1.PWM9
- net MOTOR2_PWM: now also MOTORS.3, U$1.27; no longer MOTORS.6, U$1.28
Changed lines of the file:
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@@
 <part name="GND18" library="supply1" deviceset="GND" device=""/>
 <part name="U1" library="custom" deviceset="LM555CM" device="" value="TLC555"/>
-<part name="C2" library="rcl" deviceset="C-EU" device="C0603" value="0.01uF"/>
+<part name="C2" library="rcl" deviceset="C-EU" device="C0603" value="0.1uF"/>
 <part name="RA" library="rcl" deviceset="R-EU_" device="R0603" value="330K"/>
 <part name="RB" library="rcl" deviceset="R-EU_" device="R0603" value="3.3K"/>
@@
 </segment>
 </net>
-<net name="MOTOR2_DIR" class="0">
+<net name="MOTOR1_DIR" class="0">
 <segment>
 <wire x1="-7.62" y1="104.14" x2="-7.62" y2="0" width="0.1524" layer="91"/>
@@
 </segment>
 </net>
-<net name="MOTOR1_DIR" class="0">
+<net name="MOTOR2_DIR" class="0">
 <segment>
 <wire x1="-5.08" y1="101.6" x2="-5.08" y2="12.7" width="0.1524" layer="91"/>
@@
 </segment>
 </net>
-<net name="MOTOR1_PWM" class="0">
+<net name="MOTOR2_BREAK" class="0">
 <segment>
 <pinref part="MOTORS" gate="G$1" pin="1"/>
@@
 </segment>
 </net>
-<net name="MOTOR1_BREAK" class="0">
+<net name="MOTOR2_PWM" class="0">
 <segment>
 <wire x1="86.36" y1="10.16" x2="38.1" y2="10.16" width="0.1524" layer="91"/>
@@
 </segment>
 </net>
-<net name="MOTOR2_PWM" class="0">
+<net name="MOTOR1_BREAK" class="0">
 <segment>
 <pinref part="MOTORS" gate="G$1" pin="6"/>
@@
 </segment>
 </net>
-<net name="MOTOR2_BREAK" class="0">
+<net name="MOTOR1_PWM" class="0">
 <segment>
 <pinref part="MOTORS" gate="G$1" pin="8"/>
