File: Eagle/Elec 2014/Motors Board.brd (EAGLE design)
At the start: 110 x 65 mm, 43 parts, among them IC1 LM18200T, IC2 LM18200T

Commit message: Reorganise projects & cleanup
Parts:
- R10, R5: value 470 -> 10k
- R11, R12, R13, R2, R3, R4: value 1k -> 68
- R7, R8: value 10k -> 1k
Changed lines of the file:
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@@
 <attribute name="VALUE" x="40.145" y="11.185" size="1.27" layer="27" rot="R270"/>
 </element>
-<element name="R2" library="rcl" package="R0603" value="1k" x="62" y="58" smashed="yes"/>
-<element name="R3" library="rcl" package="R0603" value="1k" x="62" y="55" smashed="yes"/>
-<element name="R4" library="rcl" package="R0603" value="1k" x="62" y="52" smashed="yes"/>
-<element name="R8" library="rcl" package="R0603" value="10k" x="87" y="44" smashed="yes" rot="R180"/>
+<element name="R2" library="rcl" package="R0603" value="68" x="62" y="58" smashed="yes"/>
+<element name="R3" library="rcl" package="R0603" value="68" x="62" y="55" smashed="yes"/>
+<element name="R4" library="rcl" package="R0603" value="68" x="62" y="52" smashed="yes"/>
+<element name="R8" library="rcl" package="R0603" value="1k" x="87" y="44" smashed="yes" rot="R180"/>
 <element name="R9" library="rcl" package="R0603" value="10k" x="83" y="44" smashed="yes"/>
-<element name="R10" library="rcl" package="R0603" value="470" x="96" y="44" smashed="yes" rot="R180"/>
+<element name="R10" library="rcl" package="R0603" value="10k" x="96" y="44" smashed="yes" rot="R180"/>
 <element name="5V_REG" library="v-reg" package="SOT223" value="MIC5239" x="50.45" y="12.39" smashed="yes" rot="R180"/>
-<element name="R5" library="rcl" package="R0603" value="470" x="13" y="44" smashed="yes" rot="R180"/>
+<element name="R5" library="rcl" package="R0603" value="10k" x="13" y="44" smashed="yes" rot="R180"/>
 <element name="R6" library="rcl" package="R0603" value="10k" x="1" y="44" smashed="yes"/>
-<element name="R7" library="rcl" package="R0603" value="10k" x="5" y="44" smashed="yes" rot="R180"/>
-<element name="R11" library="rcl" package="R0603" value="1k" x="32" y="55" smashed="yes" rot="R180"/>
-<element name="R12" library="rcl" package="R0603" value="1k" x="32" y="52" smashed="yes" rot="R180"/>
-<element name="R13" library="rcl" package="R0603" value="1k" x="32" y="58" smashed="yes" rot="R180"/>
+<element name="R7" library="rcl" package="R0603" value="1k" x="5" y="44" smashed="yes" rot="R180"/>
+<element name="R11" library="rcl" package="R0603" value="68" x="32" y="55" smashed="yes" rot="R180"/>
+<element name="R12" library="rcl" package="R0603" value="68" x="32" y="52" smashed="yes" rot="R180"/>
+<element name="R13" library="rcl" package="R0603" value="68" x="32" y="58" smashed="yes" rot="R180"/>
 <element name="C9" library="rcl" package="C0603" value="10nF" x="16.714346875" y="19.196878125" smashed="yes" rot="MR0"/>
 <element name="C10" library="rcl" package="C0603" value="10nF" x="1.42296875" y="19.139553125" smashed="yes" rot="MR180"/>

Commit message: Small fixes after testing cards
Connections:
- net N$10 renamed DIR1_
- net N$11 renamed BREAK1_
- net N$14 renamed PWM2
- net N$15 renamed BREAK2
- net N$16 renamed DIR2
- net N$17 renamed DIR2_
- net N$18 renamed PWM2_
- net N$19 renamed BREAK2_
- net N$23 renamed DIR1
- net N$24 renamed BREAK1
- net N$25 renamed PWM1
- net N$8 renamed PWM1_
Changed lines of the file:
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@@
 <wire x1="2.265678125" y1="19.14684375" x2="2.265678125" y2="21.638078125" width="1.016" layer="16"/>
 </signal>
-<signal name="N$8">
+<signal name="PWM1_">
 <contactref element="R2" pad="1"/>
 <contactref element="CTRL" pad="P$1"/>
@@
 <wire x1="96.365" y1="58.635" x2="96.365" y2="56.0734" width="0.4064" layer="1"/>
 </signal>
-<signal name="N$10">
+<signal name="DIR1_">
 <contactref element="R3" pad="1"/>
 <contactref element="CTRL" pad="P$2"/>
@@
 <wire x1="59.15" y1="53" x2="61.15" y2="55" width="0.4064" layer="1"/>
 </signal>
-<signal name="N$11">
+<signal name="BREAK1_">
 <contactref element="R4" pad="1"/>
 <contactref element="CTRL" pad="P$3"/>
@@
 <wire x1="68.85" y1="58" x2="62.85" y2="52" width="0.4064" layer="1"/>
 </signal>
-<signal name="N$23">
+<signal name="DIR1">
 <contactref element="R8" pad="1"/>
 <contactref element="IC1" pad="3"/>
@@
 <wire x1="86" y1="16.653415625" x2="85.907384375" y2="16.5608" width="0.4064" layer="16"/>
 </signal>
-<signal name="N$24">
+<signal name="BREAK1">
 <contactref element="IC1" pad="4"/>
 <contactref element="R9" pad="1"/>
@@
 <wire x1="82.15" y1="38.65" x2="82.15" y2="44" width="0.4064" layer="1"/>
 </signal>
-<signal name="N$25">
+<signal name="PWM1">
 <contactref element="IC1" pad="5"/>
 <contactref element="R10" pad="1"/>
@@
 <wire x1="96.85" y1="37.85" x2="96.85" y2="44" width="0.4064" layer="1"/>
 </signal>
-<signal name="N$14">
+<signal name="PWM2">
 <contactref element="R5" pad="1"/>
 <contactref element="IC2" pad="5"/>
@@
 <wire x1="13.6455125" y1="44.2044875" x2="13.6455125" y2="50.109234375" width="0.4064" layer="1"/>
 </signal>
-<signal name="N$15">
+<signal name="BREAK2">
 <contactref element="IC2" pad="4"/>
 <contactref element="R6" pad="1"/>
@@
 <wire x1="0.15" y1="35.15" x2="0.15" y2="44" width="0.4064" layer="1"/>
 </signal>
-<signal name="N$16">
+<signal name="DIR2">
 <contactref element="R7" pad="1"/>
 <contactref element="IC2" pad="3"/>
@@
 <wire x1="5.85" y1="47.35" x2="5.85" y2="44" width="0.4064" layer="1"/>
 </signal>
-<signal name="N$17">
+<signal name="DIR2_">
 <contactref element="R11" pad="1"/>
 <contactref element="CTRL" pad="P$7"/>
@@
 <wire x1="34.85" y1="53" x2="32.85" y2="55" width="0.4064" layer="1"/>
 </signal>
-<signal name="N$18">
+<signal name="PWM2_">
 <contactref element="R12" pad="1"/>
 <contactref element="CTRL" pad="P$6"/>
@@
 <wire x1="33.25" y1="51.6" x2="32.85" y2="52" width="0.4064" layer="1"/>
 </signal>
-<signal name="N$19">
+<signal name="BREAK2_">
 <contactref element="R13" pad="1"/>
 <contactref element="CTRL" pad="P$8"/>
